File: Barometer.kicad_sch (KiCad schematic)
At the start: 6 parts, among them J21 Conn_01x02, U6 BMP280

Commit message: I guess I made some changes
Parts:
- renumbered C21 to C1, C22 to C2, J21 to J1, R9 to R1, R10 to R2, U6 to U1
Changed lines of the file:
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@@
   (symbol (lib_id "power:+3V3") (at 201.93 115.57 0) (unit 1)
     (in_bom yes) (on_board yes)
-    (property "Reference" "#PWR038" (id 0) (at 201.93 119.38 0)
+    (property "Reference" "#PWR05" (id 0) (at 201.93 119.38 0)
       (effects (font (size 1.27 1.27)) hide)
     )
@@
   (symbol (lib_id "Device:R_Small") (at 207.01 118.11 270) (unit 1)
     (in_bom yes) (on_board yes)
-    (property "Reference" "R9" (id 0) (at 207.01 115.57 90))
+    (property "Reference" "R1" (id 0) (at 207.01 115.57 90))
     (property "Value" "2k2" (id 1) (at 207.01 118.11 90))
     (property "Footprint" "Resistor_SMD:R_0402_1005Metric" (id 2) (at 207.01 118.11 0)
@@
   (symbol (lib_id "Device:R_Small") (at 207.01 123.19 270) (unit 1)
     (in_bom yes) (on_board yes)
-    (property "Reference" "R10" (id 0) (at 207.01 120.65 90))
+    (property "Reference" "R2" (id 0) (at 207.01 120.65 90))
     (property "Value" "2k2" (id 1) (at 207.01 123.19 90))
     (property "Footprint" "Resistor_SMD:R_0402_1005Metric" (id 2) (at 207.01 123.19 0)
@@
   (symbol (lib_id "power:+3V3") (at 200.66 96.52 0) (unit 1)
     (in_bom yes) (on_board yes)
-    (property "Reference" "#PWR035" (id 0) (at 200.66 100.33 0)
+    (property "Reference" "#PWR02" (id 0) (at 200.66 100.33 0)
       (effects (font (size 1.27 1.27)) hide)
     )
@@
   (symbol (lib_id "Device:C_Small") (at 208.28 99.06 0) (unit 1)
     (in_bom yes) (on_board yes)
-    (property "Reference" "C22" (id 0) (at 210.6168 97.8916 0)
+    (property "Reference" "C2" (id 0) (at 210.6168 97.8916 0)
       (effects (font (size 1.27 1.27)) (justify left))
     )
@@
   (symbol (lib_id "Device:C_Small") (at 200.66 99.06 0) (unit 1)
     (in_bom yes) (on_board yes)
-    (property "Reference" "C21" (id 0) (at 202.9968 97.8916 0)
+    (property "Reference" "C1" (id 0) (at 202.9968 97.8916 0)
       (effects (font (size 1.27 1.27)) (justify left))
     )
@@
   (symbol (lib_id "power:GND") (at 200.66 101.6 0) (unit 1)
     (in_bom yes) (on_board yes)
-    (property "Reference" "#PWR036" (id 0) (at 200.66 107.95 0)
+    (property "Reference" "#PWR03" (id 0) (at 200.66 107.95 0)
       (effects (font (size 1.27 1.27)) hide)
     )
@@
   (symbol (lib_id "power:+3V3") (at 173.99 110.49 0) (unit 1)
     (in_bom yes) (on_board yes)
-    (property "Reference" "#PWR037" (id 0) (at 173.99 114.3 0)
+    (property "Reference" "#PWR04" (id 0) (at 173.99 114.3 0)
       (effects (font (size 1.27 1.27)) hide)
     )
@@
   (symbol (lib_id "power:GND") (at 176.53 128.27 0) (unit 1)
     (in_bom yes) (on_board yes)
-    (property "Reference" "#PWR040" (id 0) (at 176.53 134.62 0)
+    (property "Reference" "#PWR07" (id 0) (at 176.53 134.62 0)
       (effects (font (size 1.27 1.27)) hide)
     )
@@
   (symbol (lib_id "Sensor_Pressure:BMP280") (at 173.99 120.65 0) (unit 1)
     (in_bom yes) (on_board yes)
-    (property "Reference" "U6" (id 0) (at 179.832 118.2116 0)
+    (property "Reference" "U1" (id 0) (at 179.832 118.2116 0)
       (effects (font (size 1.27 1.27)) (justify left))
     )
@@
   (symbol (lib_id "power:+3V3") (at 149.86 120.65 0) (unit 1)
     (in_bom yes) (on_board yes)
-    (property "Reference" "#PWR039" (id 0) (at 149.86 124.46 0)
+    (property "Reference" "#PWR06" (id 0) (at 149.86 124.46 0)
       (effects (font (size 1.27 1.27)) hide)
     )
@@
   (symbol (lib_id "Connector_Generic:Conn_01x02") (at 200.66 134.62 0) (unit 1)
     (in_bom yes) (on_board yes) (fields_autoplaced)
-    (property "Reference" "J21" (id 0) (at 202.692 134.9815 0)
+    (property "Reference" "J1" (id 0) (at 202.692 134.9815 0)
       (effects (font (size 1.27 1.27)) (justify left))
     )
