File: Connectors.kicad_sch (KiCad schematic)
At the start: 17 parts, among them J1 Conn_01x04, J10 Conn_01x02, J11 Conn_01x02, J12 Conn_01x03, J13 Conn_01x03, J14 Conn_01x02, J15 Conn_01x03, J16 Conn_01x02, J17 Conn_01x03, J2 Conn_01x04, J3 Conn_01x03, J4 USB_B_Micro, J5 Conn_01x08, J6 Conn_01x08, J7 Conn_01x04, J8 Conn_01x04, J9 Conn_01x04

Commit message: I guess I made some changes
Parts:
- renumbered J9 to J10, J10 to J11, J11 to J12, J12 to J13, J13 to J14, J14 to J15, J15 to J16, J16 to J17, J17 to J18, J1 to J2, J2 to J3, J3 to J4, J4 to J5, J5 to J6, J6 to J7, J7 to J8, J8 to J9
