File: Gyro.kicad_sch (KiCad schematic)
At the start: 5 parts, among them J20 Conn_01x04, U5 MPU-6000

Commit message: I guess I made some changes
Parts:
- renumbered C18 to C3, C19 to C4, C20 to C5, J20 to J19, U5 to U3
Changed lines of the file:
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@@
   (symbol (lib_id "power:GND") (at 181.61 124.46 0) (unit 1)
     (in_bom yes) (on_board yes)
-    (property "Reference" "#PWR034" (id 0) (at 181.61 130.81 0)
+    (property "Reference" "#PWR044" (id 0) (at 181.61 130.81 0)
       (effects (font (size 1.27 1.27)) hide)
     )
@@
   (symbol (lib_id "power:GND") (at 199.39 119.38 0) (unit 1)
     (in_bom yes) (on_board yes)
-    (property "Reference" "#PWR033" (id 0) (at 199.39 125.73 0)
+    (property "Reference" "#PWR043" (id 0) (at 199.39 125.73 0)
       (effects (font (size 1.27 1.27)) hide)
     )
@@
   (symbol (lib_id "Device:C_Small") (at 199.39 116.84 0) (unit 1)
     (in_bom yes) (on_board yes)
-    (property "Reference" "C20" (id 0) (at 196.85 119.38 0)
+    (property "Reference" "C5" (id 0) (at 196.85 119.38 0)
       (effects (font (size 1.27 1.27)) (justify left))
     )
@@
   (symbol (lib_id "Device:C_Small") (at 205.74 111.76 90) (unit 1)
     (in_bom yes) (on_board yes)
-    (property "Reference" "C19" (id 0) (at 209.55 110.49 90)
+    (property "Reference" "C4" (id 0) (at 209.55 110.49 90)
       (effects (font (size 1.27 1.27)) (justify left))
     )
@@
   (symbol (lib_id "power:GND") (at 210.82 115.57 0) (unit 1)
     (in_bom yes) (on_board yes)
-    (property "Reference" "#PWR032" (id 0) (at 210.82 121.92 0)
+    (property "Reference" "#PWR042" (id 0) (at 210.82 121.92 0)
       (effects (font (size 1.27 1.27)) hide)
     )
@@
   (symbol (lib_id "power:GND") (at 163.83 114.3 0) (unit 1)
     (in_bom yes) (on_board yes)
-    (property "Reference" "#PWR031" (id 0) (at 163.83 120.65 0)
+    (property "Reference" "#PWR041" (id 0) (at 163.83 120.65 0)
       (effects (font (size 1.27 1.27)) hide)
     )
@@
   (symbol (lib_id "Sensor_Motion:MPU-6000") (at 181.61 106.68 0) (unit 1)
     (in_bom yes) (on_board yes)
-    (property "Reference" "U5" (id 0) (at 193.04 92.71 0))
+    (property "Reference" "U3" (id 0) (at 193.04 92.71 0))
     (property "Value" "MPU-6000" (id 1) (at 172.72 92.71 0))
     (property "Footprint" "Sensor_Motion:InvenSense_QFN-24_4x4mm_P0.5mm" (id 2) (at 181.61 127 0)
@@
   (symbol (lib_id "power:GND") (at 198.12 88.9 0) (unit 1)
     (in_bom yes) (on_board yes)
-    (property "Reference" "#PWR030" (id 0) (at 198.12 95.25 0)
+    (property "Reference" "#PWR040" (id 0) (at 198.12 95.25 0)
       (effects (font (size 1.27 1.27)) hide)
     )
@@
   (symbol (lib_id "Device:C_Small") (at 187.96 88.9 90) (unit 1)
     (in_bom yes) (on_board yes)
-    (property "Reference" "C18" (id 0) (at 191.77 87.63 90)
+    (property "Reference" "C3" (id 0) (at 191.77 87.63 90)
       (effects (font (size 1.27 1.27)) (justify left))
     )
@@
   (symbol (lib_id "Connector_Generic:Conn_01x04") (at 224.79 99.06 0) (unit 1)
     (in_bom yes) (on_board yes) (fields_autoplaced)
-    (property "Reference" "J20" (id 0) (at 226.822 99.4215 0)
+    (property "Reference" "J19" (id 0) (at 226.822 99.4215 0)
       (effects (font (size 1.27 1.27)) (justify left))
     )
@@
   (symbol (lib_id "power:+3V3_GYRO") (at 181.61 88.9 0) (unit 1)
     (in_bom yes) (on_board yes) (fields_autoplaced)
-    (property "Reference" "#PWR0132" (id 0) (at 181.61 92.71 0)
+    (property "Reference" "#PWR039" (id 0) (at 181.61 92.71 0)
       (effects (font (size 1.27 1.27)) hide)
     )
