File: MCU.kicad_sch (KiCad schematic)
At the start: 44 parts, among them Q1 BSS138, SW1 SW_Push, U10 STM32F722RETx, Y2 CSTNE8M00G55Z000R0

Commit message: I guess I made some changes
Parts:
- added D9: PURPLE, LED_SMD:LED_0603_1608Metric, symbol Device:LED_Small
- added R20: 1k, Resistor_SMD:R_0402_1005Metric, symbol Device:R_Small
- renumbered C41 to C10, C42 to C11, C43 to C12, C44 to C13, C45 to C14, C46 to C15, C37 to C6, C38 to C7, C39 to C8, C40 to C9, D5 to D1, D13 to D10, D6 to D2, D7 to D3, D8 to D4, D9 to D5, D10 to D6, D11 to D7, D12 to D8, R27 to R10, R28 to R11, R29 to R12, R30 to R13, R31 to R14, R32 to R15, R33 to R16, R34 to R17, R35 to R18, R36 to R19, R37 to R21, R20 to R3, R21 to R4, R22 to R5, R23 to R6, R24 to R7, R25 to R8, R26 to R9, U10 to U4, Y2 to Y1
Connections:
- net GND: now also R20.2
- net LED_5: now reaches U4.24 (PC4)
- net LED_5: now also D9.2 (A)
- new net PURPLE: D9.1 (K), R20.1
- no-connect marks 5 -> 4
Other:
- note added: "UART Jumpers"
- moved on the sheet: C10, C11, C12, C13, C14, C15, C6, C7, C8, C9, D1, D10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
