File: OSD.kicad_sch (KiCad schematic)
At the start: 17 parts, among them J18 Conn_01x04, U7 MAX7456EUI+, Y1 27MHz

Commit message: I guess I made some changes
Parts:
- renumbered C31 to C16, C29 to C17, C30 to C18, C32 to C19, C33 to C20, C34 to C21, C35 to C22, C36 to C23, J18 to J20, R14 to R22, R15 to R23, R16 to R24, R18 to R25, R17 to R26, R19 to R27, U7 to U5, Y1 to Y2
Changed lines of the file:
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@@
   (symbol (lib_id "Device:Crystal_GND24_Small") (at 186.69 118.11 0) (unit 1)
     (in_bom yes) (on_board yes)
-    (property "Reference" "Y1" (id 0) (at 177.8 111.76 0)
+    (property "Reference" "Y2" (id 0) (at 177.8 111.76 0)
       (effects (font (size 1.27 1.27)) (justify left))
     )
@@
   (symbol (lib_id "Device:C_Small") (at 182.88 123.19 180) (unit 1)
     (in_bom yes) (on_board yes)
-    (property "Reference" "C35" (id 0) (at 179.07 121.92 0)
+    (property "Reference" "C22" (id 0) (at 179.07 121.92 0)
       (effects (font (size 1.27 1.27)) (justify right))
     )
@@
   (symbol (lib_id "Device:C_Small") (at 193.04 123.19 180) (unit 1)
     (in_bom yes) (on_board yes)
-    (property "Reference" "C36" (id 0) (at 194.31 121.92 0)
+    (property "Reference" "C23" (id 0) (at 194.31 121.92 0)
       (effects (font (size 1.27 1.27)) (justify right))
     )
@@
   (symbol (lib_id "power:GND") (at 186.69 125.73 0) (unit 1)
     (in_bom yes) (on_board yes)
-    (property "Reference" "#PWR063" (id 0) (at 186.69 132.08 0)
+    (property "Reference" "#PWR086" (id 0) (at 186.69 132.08 0)
       (effects (font (size 1.27 1.27)) hide)
     )
@@
   (symbol (lib_id "Device:R_Small") (at 195.58 118.11 270) (unit 1)
     (in_bom yes) (on_board yes)
-    (property "Reference" "R19" (id 0) (at 195.58 113.1316 90))
+    (property "Reference" "R27" (id 0) (at 195.58 113.1316 90))
     (property "Value" "589" (id 1) (at 195.58 115.443 90))
     (property "Footprint" "Resistor_SMD:R_0402_1005Metric" (id 2) (at 195.58 118.11 0)
@@
   (symbol (lib_id "Device:C_Small") (at 217.17 118.11 0) (unit 1)
     (in_bom yes) (on_board yes)
-    (property "Reference" "C32" (id 0) (at 213.36 120.65 0))
+    (property "Reference" "C19" (id 0) (at 213.36 120.65 0))
     (property "Value" "0.1uF" (id 1) (at 219.71 116.84 0))
     (property "Footprint" "Capacitor_SMD:C_0402_1005Metric" (id 2) (at 217.17 118.11 0)
@@
   (symbol (lib_id "Device:C_Small") (at 224.79 118.11 0) (unit 1)
     (in_bom yes) (on_board yes)
-    (property "Reference" "C33" (id 0) (at 222.25 120.65 0))
+    (property "Reference" "C20" (id 0) (at 222.25 120.65 0))
     (property "Value" "0.1uF" (id 1) (at 228.6 116.84 0))
     (property "Footprint" "Capacitor_SMD:C_0402_1005Metric" (id 2) (at 224.79 118.11 0)
@@
   (symbol (lib_id "Device:C_Small") (at 232.41 118.11 0) (unit 1)
     (in_bom yes) (on_board yes)
-    (property "Reference" "C34" (id 0) (at 231.14 120.65 0))
+    (property "Reference" "C21" (id 0) (at 231.14 120.65 0))
     (property "Value" "0.1uF" (id 1) (at 236.22 116.84 0))
     (property "Footprint" "Capacitor_SMD:C_0402_1005Metric" (id 2) (at 232.41 118.11 0)
@@
   (symbol (lib_id "power:+3V3") (at 217.17 115.57 0) (unit 1)
     (in_bom yes) (on_board yes)
-    (property "Reference" "#PWR061" (id 0) (at 217.17 119.38 0)
+    (property "Reference" "#PWR084" (id 0) (at 217.17 119.38 0)
       (effects (font (size 1.27 1.27)) hide)
     )
@@
   (symbol (lib_id "power:GND") (at 217.17 120.65 0) (unit 1)
     (in_bom yes) (on_board yes)
-    (property "Reference" "#PWR062" (id 0) (at 217.17 127 0)
+    (property "Reference" "#PWR085" (id 0) (at 217.17 127 0)
       (effects (font (size 1.27 1.27)) hide)
     )
@@
   (symbol (lib_id "power:GND") (at 179.07 92.71 0) (unit 1)
     (in_bom yes) (on_board yes)
-    (property "Reference" "#PWR060" (id 0) (at 179.07 99.06 0)
+    (property "Reference" "#PWR082" (id 0) (at 179.07 99.06 0)
       (effects (font (size 1.27 1.27)) hide)
     )
@@
   (symbol (lib_id "Device:R_Small") (at 176.53 90.17 270) (unit 1)
     (in_bom yes) (on_board yes)
-    (property "Reference" "R18" (id 0) (at 179.07 88.9 90)
+    (property "Reference" "R25" (id 0) (at 179.07 88.9 90)
       (effects (font (size 1.27 1.27)) (justify left))
     )
@@
   (symbol (lib_id "power:GND") (at 217.17 76.2 0) (unit 1)
     (in_bom yes) (on_board yes)
-    (property "Reference" "#PWR057" (id 0) (at 217.17 82.55 0)
+    (property "Reference" "#PWR081" (id 0) (at 217.17 82.55 0)
       (effects (font (size 1.27 1.27)) hide)
     )
@@
   (symbol (lib_id "power:+3V3") (at 226.06 69.85 0) (unit 1)
     (in_bom yes) (on_board yes)
-    (property "Reference" "#PWR056" (id 0) (at 226.06 73.66 0)
+    (property "Reference" "#PWR080" (id 0) (at 226.06 73.66 0)
       (effects (font (size 1.27 1.27)) hide)
     )
@@
   (symbol (lib_id "power:+3V3") (at 172.72 68.58 0) (unit 1)
     (in_bom yes) (on_board yes)
-    (property "Reference" "#PWR058" (id 0) (at 172.72 72.39 0)
+    (property "Reference" "#PWR079" (id 0) (at 172.72 72.39 0)
       (effects (font (size 1.27 1.27)) hide)
     )
@@
   (symbol (lib_id "power:GND") (at 215.9 105.41 0) (unit 1)
     (in_bom yes) (on_board yes)
-    (property "Reference" "#PWR059" (id 0) (at 215.9 111.76 0)
+    (property "Reference" "#PWR083" (id 0) (at 215.9 111.76 0)
       (effects (font (size 1.27 1.27)) hide)
     )
@@
   (symbol (lib_id "Device:R_Small") (at 220.98 87.63 270) (unit 1)
     (in_bom yes) (on_board yes)
-    (property "Reference" "R16" (id 0) (at 223.52 86.36 90)
+    (property "Reference" "R24" (id 0) (at 223.52 86.36 90)
       (effects (font (size 1.27 1.27)) (justify left))
     )
@@
   (symbol (lib_id "Device:R_Small") (at 220.98 82.55 270) (unit 1)
     (in_bom yes) (on_board yes)
-    (property "Reference" "R15" (id 0) (at 223.52 81.28 90)
+    (property "Reference" "R23" (id 0) (at 223.52 81.28 90)
       (effects (font (size 1.27 1.27)) (justify left))
     )
@@
   (symbol (lib_id "Device:R_Small") (at 220.98 80.01 270) (unit 1)
     (in_bom yes) (on_board yes)
-    (property "Reference" "R14" (id 0) (at 223.52 78.74 90)
+    (property "Reference" "R22" (id 0) (at 223.52 78.74 90)
       (effects (font (size 1.27 1.27)) (justify left))
     )
@@
   (symbol (lib_id "Device:C_Small") (at 234.95 95.25 270) (unit 1)
     (in_bom yes) (on_board yes)
-    (property "Reference" "C30" (id 0) (at 232.41 93.98 90))
+    (property "Reference" "C18" (id 0) (at 232.41 93.98 90))
     (property "Value" "10uF" (id 1) (at 232.41 96.52 90))
     (property "Footprint" "Capacitor_SMD:C_0402_1005Metric" (id 2) (at 234.95 95.25 0)
@@
   (symbol (lib_id "Device:C_Small") (at 240.03 92.71 270) (unit 1)
     (in_bom yes) (on_board yes)
-    (property "Reference" "C29" (id 0) (at 241.3 90.17 90))
+    (property "Reference" "C17" (id 0) (at 241.3 90.17 90))
     (property "Value" "10uF" (id 1) (at 237.49 91.44 90))
     (property "Footprint" "Capacitor_SMD:C_0402_1005Metric" (id 2) (at 240.03 92.71 0)
@@
   (symbol (lib_id "Device:R_Small") (at 245.11 92.71 270) (unit 1)
     (in_bom yes) (on_board yes)
-    (property "Reference" "R17" (id 0) (at 246.38 93.98 90)
+    (property "Reference" "R26" (id 0) (at 246.38 93.98 90)
       (effects (font (size 1.27 1.27)) (justify left))
     )
@@
   (symbol (lib_id "Device:C_Small") (at 176.53 85.09 90) (unit 1)
     (in_bom yes) (on_board yes)
-    (property "Reference" "C31" (id 0) (at 179.07 83.82 90))
+    (property "Reference" "C16" (id 0) (at 179.07 83.82 90))
     (property "Value" "0.1uF" (id 1) (at 172.72 83.82 90))
     (property "Footprint" "Capacitor_SMD:C_0402_1005Metric" (id 2) (at 176.53 85.09 0)
@@
   (symbol (lib_id "JPW_Symbols:MAX7456EUI+") (at 200.66 87.63 0) (unit 1)
     (in_bom yes) (on_board yes) (fields_autoplaced)
-    (property "Reference" "U7" (id 0) (at 200.66 60.7273 0))
+    (property "Reference" "U5" (id 0) (at 200.66 60.7273 0))
     (property "Value" "MAX7456EUI+" (id 1) (at 200.66 63.5024 0))
     (property "Footprint" "JPW_Footprints:MAX7456" (id 2) (at 200.66 87.63 0)
@@
   (symbol (lib_id "Connector_Generic:Conn_01x04") (at 260.35 105.41 0) (unit 1)
     (in_bom yes) (on_board yes) (fields_autoplaced)
-    (property "Reference" "J18" (id 0) (at 262.382 105.7715 0)
-      (effects (font (size 1.27 1.27)) (justify left))
-    )
+    (property "Reference" "J20" (id 0) (at 262.382 105.7715 0)
+      (effects (font (size 1.27 1.27)) (justify left))
+    )
