File: Power.kicad_sch (KiCad schematic)
At the start: 37 parts, among them U3 LD1086DT33TR, U4 LP2985-3.3, U8 MP4560DQ, U9 MP4560DQ

Commit message: I guess I made some changes
Parts:
- renumbered C1 to C24, C2 to C25, C3 to C26, C4 to C27, C5 to C28, C6 to C29, C7 to C30, C8 to C31, C9 to C32, C10 to C33, C11 to C34, C12 to C35, C13 to C36, C14 to C37, C15 to C38, C16 to C39, C17 to C40, D1 to D11, D2 to D12, D3 to D13, D4 to D14, FB3 to FB2, FB2 to FB3, L3 to L6, L4 to L7, R1 to R28, R2 to R29, R3 to R30, R4 to R31, R5 to R32, R6 to R33, R7 to R34, R8 to R35, U8 to U6, U9 to U7, U3 to U8, U4 to U9
