File: WormDriver.kicad_sch (KiCad schematic)
At the start: 7 parts, among them J19 Conn_01x04, U2 DRV8834RGER

Commit message: I guess I made some changes
Parts:
- renumbered C23 to C41, C24 to C42, C25 to C43, J19 to J21, R11 to R36, R12 to R37, U2 to U10
Changed lines of the file:
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@@
   (symbol (lib_id "power:+5V") (at 234.95 86.36 0) (unit 1)
     (in_bom yes) (on_board yes) (fields_autoplaced)
-    (property "Reference" "#PWR0137" (id 0) (at 234.95 90.17 0)
+    (property "Reference" "#PWR0118" (id 0) (at 234.95 90.17 0)
       (effects (font (size 1.27 1.27)) hide)
     )
@@
   (symbol (lib_id "Connector_Generic:Conn_01x04") (at 224.79 111.76 0) (unit 1)
     (in_bom yes) (on_board yes) (fields_autoplaced)
-    (property "Reference" "J19" (id 0) (at 226.822 112.1215 0)
+    (property "Reference" "J21" (id 0) (at 226.822 112.1215 0)
       (effects (font (size 1.27 1.27)) (justify left))
     )
@@
   (symbol (lib_id "power:+5V") (at 215.9 86.36 0) (unit 1)
     (in_bom yes) (on_board yes) (fields_autoplaced)
-    (property "Reference" "#PWR0135" (id 0) (at 215.9 90.17 0)
+    (property "Reference" "#PWR0116" (id 0) (at 215.9 90.17 0)
       (effects (font (size 1.27 1.27)) hide)
     )
@@
   (symbol (lib_id "power:GND") (at 190.5 115.57 0) (mirror y) (unit 1)
     (in_bom yes) (on_board yes) (fields_autoplaced)
-    (property "Reference" "#PWR0140" (id 0) (at 190.5 121.92 0)
+    (property "Reference" "#PWR0122" (id 0) (at 190.5 121.92 0)
       (effects (font (size 1.27 1.27)) hide)
     )
@@
   (symbol (lib_id "power:+5V") (at 170.18 73.66 0) (unit 1)
     (in_bom yes) (on_board yes) (fields_autoplaced)
-    (property "Reference" "#PWR0139" (id 0) (at 170.18 77.47 0)
+    (property "Reference" "#PWR0114" (id 0) (at 170.18 77.47 0)
       (effects (font (size 1.27 1.27)) hide)
     )
@@
   (symbol (lib_id "Device:C_Small") (at 193.04 82.55 90) (unit 1)
     (in_bom yes) (on_board yes)
-    (property "Reference" "C23" (id 0) (at 191.77 83.82 90)
+    (property "Reference" "C41" (id 0) (at 191.77 83.82 90)
       (effects (font (size 1.27 1.27)) (justify left))
     )
@@
   (symbol (lib_id "power:GND") (at 147.32 105.41 0) (unit 1)
     (in_bom yes) (on_board yes)
-    (property "Reference" "#PWR0141" (id 0) (at 147.32 111.76 0)
+    (property "Reference" "#PWR0120" (id 0) (at 147.32 111.76 0)
       (effects (font (size 1.27 1.27)) hide)
     )
@@
   (symbol (lib_id "Device:R_Small") (at 226.06 88.9 180) (unit 1)
     (in_bom yes) (on_board yes)
-    (property "Reference" "R11" (id 0) (at 228.6 88.9 0))
+    (property "Reference" "R36" (id 0) (at 228.6 88.9 0))
     (property "Value" "47k" (id 1) (at 223.52 88.9 0))
     (property "Footprint" "Resistor_SMD:R_0402_1005Metric" (id 2) (at 226.06 88.9 0)
@@
   (symbol (lib_id "power:GND") (at 152.4 123.19 0) (unit 1)
     (in_bom yes) (on_board yes) (fields_autoplaced)
-    (property "Reference" "#PWR0143" (id 0) (at 152.4 129.54 0)
+    (property "Reference" "#PWR0123" (id 0) (at 152.4 129.54 0)
       (effects (font (size 1.27 1.27)) hide)
     )
@@
   (symbol (lib_id "power:GND") (at 171.45 129.54 0) (unit 1)
     (in_bom yes) (on_board yes) (fields_autoplaced)
-    (property "Reference" "#PWR0142" (id 0) (at 171.45 135.89 0)
+    (property "Reference" "#PWR0124" (id 0) (at 171.45 135.89 0)
       (effects (font (size 1.27 1.27)) hide)
     )
@@
   (symbol (lib_id "power:+5V") (at 226.06 86.36 0) (unit 1)
     (in_bom yes) (on_board yes) (fields_autoplaced)
-    (property "Reference" "#PWR0136" (id 0) (at 226.06 90.17 0)
+    (property "Reference" "#PWR0117" (id 0) (at 226.06 90.17 0)
       (effects (font (size 1.27 1.27)) hide)
     )
@@
   (symbol (lib_id "Device:C_Small") (at 193.04 107.95 90) (unit 1)
     (in_bom yes) (on_board yes)
-    (property "Reference" "C25" (id 0) (at 191.77 109.22 90)
+    (property "Reference" "C43" (id 0) (at 191.77 109.22 90)
       (effects (font (size 1.27 1.27)) (justify left))
     )
@@
   (symbol (lib_id "power:+5V") (at 198.12 80.01 0) (unit 1)
     (in_bom yes) (on_board yes) (fields_autoplaced)
-    (property "Reference" "#PWR0138" (id 0) (at 198.12 83.82 0)
+    (property "Reference" "#PWR0115" (id 0) (at 198.12 83.82 0)
       (effects (font (size 1.27 1.27)) hide)
     )
@@
   (symbol (lib_id "Device:C_Polarized_Small") (at 215.9 88.9 0) (unit 1)
     (in_bom yes) (on_board yes)
-    (property "Reference" "C24" (id 0) (at 210.82 87.63 0)
+    (property "Reference" "C42" (id 0) (at 210.82 87.63 0)
       (effects (font (size 1.27 1.27)) (justify left))
     )
@@
   (symbol (lib_id "power:GND") (at 215.9 91.44 0) (mirror y) (unit 1)
     (in_bom yes) (on_board yes) (fields_autoplaced)
-    (property "Reference" "#PWR0134" (id 0) (at 215.9 97.79 0)
+    (property "Reference" "#PWR0119" (id 0) (at 215.9 97.79 0)
       (effects (font (size 1.27 1.27)) hide)
     )
@@
   (symbol (lib_id "JPW_Symbols:DRV8834RGER") (at 171.45 102.87 0) (unit 1)
     (in_bom yes) (on_board yes) (fields_autoplaced)
-    (property "Reference" "U2" (id 0) (at 173.5951 127.4457 0)
+    (property "Reference" "U10" (id 0) (at 173.5951 127.4457 0)
       (effects (font (size 1.524 1.524)) (justify left))
     )
@@
   (symbol (lib_id "Device:R_Small") (at 234.95 88.9 180) (unit 1)
     (in_bom yes) (on_board yes)
-    (property "Reference" "R12" (id 0) (at 237.49 88.9 0))
+    (property "Reference" "R37" (id 0) (at 237.49 88.9 0))
     (property "Value" "47k" (id 1) (at 232.41 88.9 0))
     (property "Footprint" "Resistor_SMD:R_0402_1005Metric" (id 2) (at 234.95 88.9 0)
@@
   (symbol (lib_id "power:GND") (at 198.12 110.49 0) (mirror y) (unit 1)
     (in_bom yes) (on_board yes) (fields_autoplaced)
-    (property "Reference" "#PWR0133" (id 0) (at 198.12 116.84 0)
-      (effects (font (size 1.27 1.27)) hide)
-    )
+    (property "Reference" "#PWR0121" (id 0) (at 198.12 116.84 0)
+      (effects (font (size 1.27 1.27)) hide)
+    )
