File: Autodrone_V2.kicad_pcb (KiCad board)
At the start: 6 copper layers, 54.8 x 39.2 mm, 143 parts, among them J1 Conn_01x04, J10 Conn_01x02, J11 Conn_01x02, J12 Conn_01x03, J13 Conn_01x03, J14 Conn_01x02, J15 Conn_01x03, J16 Conn_01x02, J17 Conn_01x03, J18 Conn_01x04, J19 Conn_01x04, J2 Conn_01x04, J20 Conn_01x04, J21 Conn_01x02, J3 Conn_01x03, J4 USB_B_Micro, J5 Conn_01x08, J6 Conn_01x08, J7 Conn_01x04, J8 Conn_01x04, J9 Conn_01x04, Q1 BSS138, SW1 SW_Push, U1 STLINK-V3MODS, U10 STM32F722RETx, U2 DRV8834RGER, U3 LD1086DT33TR, U4 LP2985-3.3, U5 MPU-6000, U6 BMP280, U7 MAX7456EUI+, U8 MP4560DQ, U9 MP4560DQ, Y1 27MHz, Y2 CSTNE8M00G55Z000R0

Commit message: I guess I made some changes
Parts:
- added D9: PURPLE, LED_SMD:LED_0603_1608Metric, F.Cu at (72.1, 78.6)
- added R20: 1k, Resistor_SMD:R_0402_1005Metric, B.Cu at (71.7, 78.2)
- moved L5 5.35 mm to (115.0, 94.8), turned to 90 degrees
- moved D3 0.71 mm to (75.2, 75.5)
- moved D5 0.71 mm to (74.2, 76.5)
- moved D7 0.71 mm to (73.1, 77.5)
- moved R10 0.71 mm to (75.9, 74.1)
- moved R16 0.71 mm to (73.8, 76.1)
- moved R18 0.71 mm to (72.8, 77.2)
- moved R14 0.71 mm to (74.8, 75.1)
- moved D1 0.71 mm to (76.2, 74.4)
- moved L3 0.26 mm to (76.9, 79.2)
- renumbered C21 to C1, C41 to C10, C42 to C11, C43 to C12, C44 to C13, C45 to C14, C46 to C15, C31 to C16, C29 to C17, C30 to C18, C32 to C19, C22 to C2, C33 to C20, C34 to C21, C35 to C22, C36 to C23, C1 to C24, C2 to C25, C3 to C26, C4 to C27, C5 to C28, C6 to C29, C18 to C3, C7 to C30, C8 to C31, C9 to C32, C10 to C33, C11 to C34, C12 to C35, C13 to C36, C14 to C37, C15 to C38, C16 to C39, C19 to C4, C17 to C40, C23 to C41, C24 to C42, C25 to C43, C20 to C5, C37 to C6, C38 to C7, C39 to C8, C40 to C9, D5 to D1, D13 to D10, D1 to D11, D2 to D12, D3 to D13, D4 to D14, D6 to D2, D7 to D3, D8 to D4, D9 to D5, D10 to D6, D11 to D7, D12 to D8, FB3 to FB2, FB2 to FB3, J21 to J1, J9 to J10, J10 to J11, J11 to J12, J12 to J13, J13 to J14, J14 to J15, J15 to J16, J16 to J17, J17 to J18, J20 to J19, J1 to J2, J18 to J20, J19 to J21, J2 to J3, J3 to J4, J4 to J5, J5 to J6, J6 to J7, J7 to J8, J8 to J9, L5 to L3, L6 to L4, L7 to L5, L3 to L6, L4 to L7, R9 to R1, R27 to R10, R28 to R11, R29 to R12, R30 to R13, R31 to R14, R32 to R15, R33 to R16, R34 to R17, R35 to R18, R36 to R19, R10 to R2, R37 to R21, R14 to R22, R15 to R23, R16 to R24, R18 to R25, R17 to R26, R19 to R27, R1 to R28, R2 to R29, R20 to R3, R3 to R30, R4 to R31, R5 to R32, R6 to R33, R7 to R34, R8 to R35, R11 to R36, R12 to R37, R21 to R4, R22 to R5, R23 to R6, R24 to R7, R25 to R8, R26 to R9, U6 to U1, U2 to U10, U1 to U2, U5 to U3, U10 to U4, U7 to U5, U8 to U6, U9 to U7, U3 to U8, U4 to U9, Y2 to Y1, Y1 to Y2
Connections:
- U4 pad 24: unconnected-(U10-Pad24) -> /MCU/LED_5
Routing:
- net /MCU/LED_5: track 0.00 -> 40.8 mm, vias 0 -> 3
- net /MCU/PURPLE: track 0.00 -> 1.20 mm, vias 0 -> 1
- net /WormDriver/VREF: track 1.00 -> 0.00 mm
- net GND: vias 87 -> 88
- added copper zone on B.Cu, net /WormDriver/VREF
Other:
- board text added: "5 4 3 2 1"
- board text added: "JUMPER"
- board text removed: "4 3 2 1"
- board text removed: "JUMP"

Commit message: Added new files
Other:
- rule pad_to_mask_clearance: 0.0508 -> 0
Changed lines of the file:
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@@
       (edge_plating yes)
     )
-    (pad_to_mask_clearance 0.0508)
+    (pad_to_mask_clearance 0)
     (pcbplotparams
       (layerselection 0x00010fc_ffffffff)
@@
     (pad "1" smd roundrect (at -3.5 -2 90) (size 0.6 1.55) (layers "F.Cu" "F.Paste" "F.Mask") (roundrect_rratio 0.25)
       (net 4 "VCC") (pinfunction "Pin_1") (pintype "passive"))
-    (pad "2" smd roundrect (at -4.8 1.875 90) (size 1.2 1.8) (layers "F.Cu" "F.Paste" "F.Mask") (roundrect_rratio 0.208333)
+    (pad "2" smd roundrect (at -4.8 1.875 90) (size 1.2 1.8) (layers "F.Cu" "F.Paste" "F.Mask") (roundrect_rratio 0.2083333333)
       (net 1 "GND") (pinfunction "Pin_2") (pintype "passive"))
-    (pad "2" smd roundrect (at 4.8 1.875 90) (size 1.2 1.8) (layers "F.Cu" "F.Paste" "F.Mask") (roundrect_rratio 0.208333)
+    (pad "2" smd roundrect (at 4.8 1.875 90) (size 1.2 1.8) (layers "F.Cu" "F.Paste" "F.Mask") (roundrect_rratio 0.2083333333)
       (net 1 "GND") (pinfunction "Pin_2") (pintype "passive"))
     (pad "2" smd roundrect (at -2.5 -2 90) (size 0.6 1.55) (layers "F.Cu" "F.Paste" "F.Mask") (roundrect_rratio 0.25)
@@
     (fp_circle (center 2.1 0) (end 2.95 0) (layer "F.Fab") (width 0.1) (fill none))
     (fp_circle (center -2.1 0) (end -1.25 0) (layer "F.Fab") (width 0.1) (fill none))
-    (pad "1" thru_hole roundrect (at -2.1 0 225) (size 1.85 1.85) (drill 0.85) (layers *.Cu *.Mask) (roundrect_rratio 0.135135)
+    (pad "1" thru_hole roundrect (at -2.1 0 225) (size 1.85 1.85) (drill 0.85) (layers *.Cu *.Mask) (roundrect_rratio 0.1351351351)
       (net 53 "/WORM2_L") (pinfunction "Pin_1") (pintype "passive"))
     (pad "2" thru_hole circle (at 2.1 0 225) (size 1.85 1.85) (drill 0.85) (layers *.Cu *.Mask)
@@
     (fp_circle (center -2.1 0) (end -1.25 0) (layer "F.Fab") (width 0.1) (fill none))
     (fp_circle (center 2.1 0) (end 2.95 0) (layer "F.Fab") (width 0.1) (fill none))
-    (pad "1" thru_hole roundrect (at -2.1 0 315) (size 1.85 1.85) (drill 0.85) (layers *.Cu *.Mask) (roundrect_rratio 0.135135)
+    (pad "1" thru_hole roundrect (at -2.1 0 315) (size 1.85 1.85) (drill 0.85) (layers *.Cu *.Mask) (roundrect_rratio 0.1351351351)
       (net 55 "/WORM1_H") (pinfunction "Pin_1") (pintype "passive"))
     (pad "2" thru_hole circle (at 2.1 0 315) (size 1.85 1.85) (drill 0.85) (layers *.Cu *.Mask)
@@
       (effects (font (size 0.787402 0.787402) (thickness 0.15)))
     )
-    (fp_text user "32" (at 8.509 11.1252 90) (layer "F.Fab")
+    (fp_text user "17" (at 8.89 29.972 90) (layer "F.Fab")
       (effects (font (size 1.18 1.18) (thickness 0.15)))
     )
-    (fp_text user "1" (at -9.652 10.668 90) (layer "F.Fab")
+    (fp_text user "32" (at 8.509 11.1252 90) (layer "F.Fab")
       (effects (font (size 1.18 1.18) (thickness 0.15)))
     )
@@
       (effects (font (size 1.18 1.18) (thickness 0.15)))
     )
-    (fp_text user "17" (at 8.89 29.972 90) (layer "F.Fab")
+    (fp_text user "1" (at -9.652 10.668 90) (layer "F.Fab")
       (effects (font (size 1.18 1.18) (thickness 0.15)))
     )
-    (fp_line (start -7.62 29.972) (end -7.62 29.6672) (layer "F.SilkS") (width 0.1524))
-    (fp_line (start -7.62 9.1948) (end -7.62 0) (layer "F.SilkS") (width 0.1524))
-    (fp_line (start 7.62 9.1948) (end 7.62 0) (layer "F.SilkS") (width 0.1524))
     (fp_line (start -4.8006 -1.0922) (end 4.8006 -1.0922) (layer "F.SilkS") (width 0.1524))
-    (fp_line (start 7.62 29.972) (end 7.62 29.6672) (layer "F.SilkS") (width 0.1524))
-    (fp_line (start -7.62 29.972) (end 7.62 29.972) (layer "F.SilkS") (width 0.1524))
     (fp_line (start 5.8928 0) (end 7.62 0) (layer "F.SilkS") (width 0.1524))
+    (fp_line (start -7.62 29.972) (end 7.62 29.972) (layer "F.SilkS") (width 0.1524))
+    (fp_line (start -7.62 29.972) (end -7.62 29.6672) (layer "F.SilkS") (width 0.1524))
     (fp_line (start -7.62 0) (end -5.8928 0) (layer "F.SilkS") (width 0.1524))
+    (fp_line (start 7.62 29.972) (end 7.62 29.6672) (layer "F.SilkS") (width 0.1524))
+    (fp_line (start 7.62 9.1948) (end 7.62 0) (layer "F.SilkS") (width 0.1524))
+    (fp_line (start -7.62 9.1948) (end -7.62 0) (layer "F.SilkS") (width 0.1524))
     (fp_arc (start 5.8928 0) (mid 5.120498 -0.319898) (end 4.8006 -1.0922) (layer "F.SilkS") (width 0.1524))
     (fp_arc (start -4.8006 -1.0922) (mid -5.120498 -0.319898) (end -5.8928 0) (layer "F.SilkS") (width 0.1524))
-    (fp_line (start 8.69 -2.17) (end 8.69 31.05) (layer "F.CrtYd") (width 0.12))
-    (fp_line (start -9.27 -2.17) (end -9.27 31.05) (layer "F.CrtYd") (width 0.12))
     (fp_line (start -9.27 -2.17) (end 8.69 -2.17) (layer "F.CrtYd") (width 0.12))
     (fp_line (start 8.69 31.05) (end -9.27 31.05) (layer "F.CrtYd") (width 0.12))
+    (fp_line (start -9.27 -2.17) (end -9.27 31.05) (layer "F.CrtYd") (width 0.12))
+    (fp_line (start 8.69 -2.17) (end 8.69 31.05) (layer "F.CrtYd") (width 0.12))
     (pad "1" smd rect (at -7.32003 9.906 90) (size 1.89992 1.0701) (layers "F.Cu" "F.Paste" "F.Mask")
       (net 107 "unconnected-(U2-Pad1)") (pinfunction "BRIDGE_UART_RX") (pintype "passive+no_connect"))
@@
       (net 130 "unconnected-(U2-Pad32)") (pinfunction "T_SW_DIR") (pintype "passive+no_connect"))
     (model "${MY_3DMODELS}/STLINK-V3MODS.step"
-      (offset (xyz 0 0 1.5))
+      (offset (xyz 0 -30.05 -1.5))
       (scale (xyz 1 1 1))
-      (rotate (xyz 0 0 0))
+      (rotate (xyz 0 0 90))
     )
   )
@@
     (fp_line (start 2 2) (end 2 -2) (layer "B.Fab") (width 0.1))
     (fp_line (start -1 2) (end 2 2) (layer "B.Fab") (width 0.1))
-    (pad "" smd roundrect (at 0.66 0.66 180) (size 1.08 1.08) (layers "B.Paste") (roundrect_rratio 0.217391))
-    (pad "" smd roundrect (at -0.66 0.66 180) (size 1.08 1.08) (layers "B.Paste") (roundrect_rratio 0.217391))
-    (pad "" smd roundrect (at 0.66 -0.66 180) (size 1.08 1.08) (layers "B.Paste") (roundrect_rratio 0.217391))
-    (pad "" smd roundrect (at -0.66 -0.66 180) (size 1.08 1.08) (layers "B.Paste") (roundrect_rratio 0.217391))
+    (pad "" smd roundrect (at 0.66 0.66 180) (size 1.08 1.08) (layers "B.Paste") (roundrect_rratio 0.2173907407))
+    (pad "" smd roundrect (at -0.66 0.66 180) (size 1.08 1.08) (layers "B.Paste") (roundrect_rratio 0.2173907407))
+    (pad "" smd roundrect (at 0.66 -0.66 180) (size 1.08 1.08) (layers "B.Paste") (roundrect_rratio 0.2173907407))
+    (pad "" smd roundrect (at -0.66 -0.66 180) (size 1.08 1.08) (layers "B.Paste") (roundrect_rratio 0.2173907407))
     (pad "1" smd roundrect (at -1.95 1.25 180) (size 0.85 0.3) (layers "B.Cu" "B.Paste" "B.Mask") (roundrect_rratio 0.25)
       (net 55 "/WORM1_H") (pinfunction "AOUT1") (pintype "output"))
@@
     (fp_line (start 0.8 0.425) (end -0.5 0.425) (layer "B.Fab") (width 0.1))
     (fp_line (start -0.5 0.425) (end -0.8 0.125) (layer "B.Fab") (width 0.1))
-    (pad "1" smd roundrect locked (at -0.7125 0 180) (size 1.075 1.05) (layers "B.Cu" "B.Paste" "B.Mask") (roundrect_rratio 0.238095)
+    (pad "1" smd roundrect locked (at -0.7125 0 180) (size 1.075 1.05) (layers "B.Cu" "B.Paste" "B.Mask") (roundrect_rratio 0.2380952381)
       (net 5 "+5V") (pintype "passive"))
-    (pad "2" smd roundrect locked (at 0.7125 0 180) (size 1.075 1.05) (layers "B.Cu" "B.Paste" "B.Mask") (roundrect_rratio 0.238095)
+    (pad "2" smd roundrect locked (at 0.7125 0 180) (size 1.075 1.05) (layers "B.Cu" "B.Paste" "B.Mask") (roundrect_rratio 0.2380952381)
       (net 1 "GND") (pintype "passive"))
     (model "${KICAD6_3DMODEL_DIR}/Capacitor_Tantalum_SMD.3dshapes/CP_EIA-1608-08_AVX-J.wrl"
